File: PCB/FT_Hall/FT_Hall.kicad_pcb (KiCad board)
At the start: 2 copper layers, 7.6 x 19 mm, 5 parts, among them CON1 Conn_01x03_Pin

Commit message: changed hall, switch
Parts:
- C1, C2: footprint Capacitor_SMD:C_0603_1608Metric_Pad1.08x0.95mm_HandSolder -> Capacitor_SMD:C_0805_2012Metric_Pad1.18x1.45mm_HandSolder
- R1: footprint Resistor_SMD:R_0603_1608Metric_Pad0.98x0.95mm_HandSolder -> Resistor_SMD:R_0805_2012Metric_Pad1.20x1.40mm_HandSolder
- moved R1 2.18 mm to (130.8, 73.7)
- moved CON1 1.27 mm to (133.3, 68.6)
Routing:
- net /VS: track 6.99 -> 8.91 mm
- net GND: track 17.2 -> 18.6 mm
- net /Q: track 13.9 -> 15.0 mm
- net +12V: track 5.08 -> 4.08 mm
Other:
- board size 7.6 x 19 mm -> 7.6 x 19.7 mm
