File: PCB/FT_MainBoard/FT_MainBoard.kicad_pcb (KiCad board)
At the start: 2 copper layers, 110 x 75 mm, 58 parts, among them CON1 Conn_01x02_Pin, CON3 Conn_01x03, CON4 Conn_01x02_Pin, CON5 Conn_01x04_Pin, CON6 AVR-ISP-6, IC1 ATmega328PB-AU, IC2 FT231XS-R, IC3 74HC3G14DP,125, IC4 L78M05ABDT-TR, SW1 SW_Push, SW2 SW_Push, SW3 SW_Push, SW4 SW_Push, SW5 SW_SPST

Commit message: major changes, production ready
Parts:
- removed C12: 100nF, Capacitor_SMD:C_0603_1608Metric
- removed C13: 1nF, Capacitor_SMD:C_0603_1608Metric
- removed OPT1, OPT2: TLP185xSE, Package_SO:SOIC-4_4.55x3.7mm_P2.54mm
- added D1: BZX384-B5V1,115, Diode_SMD:D_SOD-323, B.Cu at (68.6, 104.6)
- added D2: BZX384-B5V1,115, Diode_SMD:D_SOD-323, B.Cu at (73.2, 104.6)
- added L: TestPoint_Pad_1.0x1.0mm, TestPoint:TestPoint_Pad_1.0x1.0mm, F.Cu at (91.0, 112.5)
- added Q1: PMBT3904,215, Package_TO_SOT_SMD:SOT-23, B.Cu at (73.2, 111.3)
- added Q2: PMBT3904,215, Package_TO_SOT_SMD:SOT-23, B.Cu at (68.6, 111.3)
- added R: TestPoint_Pad_1.0x1.0mm, TestPoint:TestPoint_Pad_1.0x1.0mm, F.Cu at (91.0, 116.5)
- added R17: 10K, Resistor_SMD:R_0603_1608Metric, B.Cu at (68.6, 106.7)
- added R18: 10K, Resistor_SMD:R_0603_1608Metric, B.Cu at (73.2, 106.7)
- added R19: 1.2K, Capacitor_SMD:C_0603_1608Metric, B.Cu at (73.2, 102.6)
- added R20: 1.2K, Capacitor_SMD:C_0603_1608Metric, B.Cu at (73.2, 101.1)
- added R21: 4K7, Resistor_SMD:R_0603_1608Metric, B.Cu at (119.9, 96.5)
- added R22: 10K, Resistor_SMD:R_0603_1608Metric, B.Cu at (119.9, 95.0)
- added RESET: TestPoint_Pad_1.0x1.0mm, TestPoint:TestPoint_Pad_1.0x1.0mm, F.Cu at (92.0, 103.5)
- added RX: TestPoint_Pad_1.0x1.0mm, TestPoint:TestPoint_Pad_1.0x1.0mm, F.Cu at (112.0, 101.7)
- added START: TestPoint_Pad_1.0x1.0mm, TestPoint:TestPoint_Pad_1.0x1.0mm, F.Cu at (89.0, 103.5)
- added STOP: TestPoint_Pad_1.0x1.0mm, TestPoint:TestPoint_Pad_1.0x1.0mm, F.Cu at (95.0, 103.5)
- added TX: TestPoint_Pad_1.0x1.0mm, TestPoint:TestPoint_Pad_1.0x1.0mm, F.Cu at (112.0, 104.6)
- C11: value 1uF -> 330nF
- C14, C15: value 100nF -> 1n
- CON3: value Conn_01x03 -> Conn_01x04_Pin; footprint custom_components:CON_3_pin -> custom_components:CON_4_pin
- R13, R14: value 550R -> 1.2K; footprint Resistor_SMD:R_0603_1608Metric -> Capacitor_SMD:C_0603_1608Metric
- moved C14 5.08 mm to (73.2, 108.2)
- moved C15 5.08 mm to (68.6, 108.2)
- moved R13 4.62 mm to (68.6, 102.6), turned to 180 degrees
- moved C11 3.00 mm to (125.2, 98.2)
- moved CON3 1.23 mm to (121.5, 80.0), turned to 90 degrees
- moved R14 0.51 mm to (68.6, 101.1), turned to 180 degrees
- moved C5 0.18 mm to (116.3, 97.3)
- moved C7 0.18 mm to (116.3, 95.8)
- moved R4 0.18 mm to (116.3, 92.7)
- moved R5 0.18 mm to (116.3, 94.2)
- moved C6 0.18 mm to (116.3, 91.2)
Connections:
- C14 pad 1: Net-(C14-Pad1) -> Net-(Q1-B)
- C15 pad 1: Net-(C15-Pad1) -> Net-(Q2-B)
- CON3 pad 1: /USB_D- -> Net-(CON3-Pin_1)
- CON3 pad 3: GND -> /USB_D-
- CON5 pad 3: /IN_LEFT -> Net-(CON5-Pin_3)
- CON5 pad 4: /IN_RIGHT -> Net-(CON5-Pin_4)
- IC1 pad 1: OPTR -> RIGHT
- IC1 pad 32: OPTL -> LEFT
- IC2 pad 17: Net-(IC2-CBUS1) -> VBUS_SENSE
- IC2 pad 19: unconnected-(IC2-CBUS3-Pad19) -> Net-(IC2-CBUS3)
- R13 pad 1: Net-(C14-Pad1) -> Net-(CON5-Pin_4)
- R13 pad 2: /IN_LEFT -> Net-(R13-Pad2)
- R14 pad 1: Net-(C15-Pad1) -> Net-(R13-Pad2)
- R14 pad 2: /IN_RIGHT -> +12V
- R3 pad 1: Net-(IC2-CBUS1) -> Net-(IC2-CBUS3)
Routing:
- net RIGHT: track 0.00 -> 47.8 mm, vias 0 -> 2
- net OPTR: track 46.6 -> 0.00 mm, vias 2 -> 0
- net LEFT: track 0.00 -> 45.4 mm, vias 0 -> 2
- net OPTL: track 44.4 -> 0.00 mm, vias 2 -> 0
- net +12V: track 87.4 -> 118.1 mm, vias 0 -> 2
- net Net-(CON5-Pin_3): track 0.00 -> 30.1 mm
- net Net-(CON5-Pin_4): track 0.00 -> 28.7 mm
- net /IN_RIGHT: track 22.8 -> 0.00 mm
- net /IN_LEFT: track 22.0 -> 0.00 mm
- net Net-(CON3-Pin_1): track 0.00 -> 19.1 mm
- net Net-(IC2-CBUS1): track 17.8 -> 0.00 mm
- net Net-(IC2-CBUS3): track 0.00 -> 16.6 mm
- net RESET: track 25.9 -> 37.0 mm
- net GND: track 9.33 -> 18.3 mm, vias 3 -> 9
- net VBUS_SENSE: track 0.00 -> 5.56 mm
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Other:
- board text added: "DTR"

Commit message: panelization
Parts:
- C1, C10, C11, C14, C15, C16, C17, C18, C2, C3, C4, C5, C6, C7, C8, C9, CON1, CON3, CON4, CON5, CON6, D1, D2, G***, IC1, IC2, IC3, IC4, LED1, LED2, LED3, OSC1, Q1, Q2, R1, R10, R11, R12, R13, R14, R15, R16, R17, R18, R19, R2, R20, R21, R22, R3, R4, R5, R6, R7, R8, R9, SW4, SW5: moved to F.Cu
- G***, HDR1, L, R, RESET, RV1, RX, START, STOP, SW1, SW2, SW3, TX: moved to B.Cu
- moved G*** 93.2 mm to (150.4, 94.0), turned to 180 degrees
- moved RV1 92.1 mm to (57.8, 109.2), turned to 0 degrees
- moved CON6 91.8 mm to (57.9, 94.5), turned to 180 degrees
- moved G*** 89.2 mm to (148.4, 109.2), turned to 0 degrees
- moved SW2 77.7 mm to (142.7, 62.0), turned to 180 degrees
- moved C15 70.5 mm to (139.1, 108.2), turned to 180 degrees
- moved Q2 70.5 mm to (139.1, 111.3)
- moved R13 70.5 mm to (139.1, 102.6), turned to 0 degrees
- moved R14 70.5 mm to (139.1, 101.1), turned to 0 degrees
- moved R17 70.5 mm to (139.1, 106.7), turned to 180 degrees
- moved D1 70.4 mm to (139.0, 104.6), turned to 0 degrees
- moved HDR1 68.3 mm to (69.7, 118.0)
- moved C14 61.4 mm to (134.5, 108.2), turned to 180 degrees
- moved D2 61.4 mm to (134.5, 104.6), turned to 180 degrees
- moved Q1 61.4 mm to (134.5, 111.3)
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
Commit message: update
Routing:
- net GND: track 18.3 -> 20.8 mm, vias 9 -> 8
Other:
- outline, holes or cut-outs redrawn
