File: PCB/FT_MainBoard/FT_MainBoard.kicad_sch (KiCad schematic)
At the start: 49 parts, among them SW1 SW_Push, SW2 SW_SPST

Commit message: final update
Parts:
- removed CON_TARGETS1: Conn_01x04_Pin, Connector_PinHeader_2.54mm:PinHeader_1x04_P2.54mm_Horizontal, symbol Connector:Conn_01x04_Pin
- removed USB1: USB_B, Connector_USB:USB_B_Lumberg_2411_02_Horizontal, symbol Connector:USB_B
- added CON2: Conn_02x08_Odd_Even, KLS_connector:16_pin, symbol Connector_Generic:Conn_02x08_Odd_Even
- added CON3: Conn_01x03, custom_components:CON_3_pin, symbol Connector_Generic:Conn_01x03
- added CON5: Conn_01x04_Pin, custom_components:CON_4_pin, symbol Connector:Conn_01x04_Pin
- added HDR1: Conn_01x16_Pin, Connector_PinHeader_2.54mm:PinHeader_1x16_P2.54mm_Vertical, symbol Connector:Conn_01x16_Pin
- added R1: 200R, Resistor_SMD:R_0603_1608Metric, symbol Device:R
- added RV1: Vishay 64X 10K, Connector_PinHeader_2.54mm:PinHeader_1x03_P2.54mm_Vertical, symbol Device:R_Potentiometer_Trim
- added SW1, SW2, SW3: SW_Push, Button_Switch_THT:SW_PUSH-12mm, symbol Switch:SW_Push
- C1: renamed from C_MCU1; Assembly (none) -> YES; Supplier (none) -> PCBWAY
- C10: renamed from C_IN3; Assembly (none) -> YES; Supplier (none) -> PCBWAY
- C11: renamed from C_VIN1; Assembly (none) -> YES; Supplier (none) -> PCBWAY
- C12: renamed from C_VIN2; Assembly (none) -> YES; Supplier (none) -> PCBWAY
- C13: renamed from C_VIN3; Assembly (none) -> YES; Supplier (none) -> PCBWAY
- C14: renamed from C_OPTL1; Assembly (none) -> YES; Supplier (none) -> PCBWAY
- C15: renamed from C_OPTR1; Assembly (none) -> YES; Supplier (none) -> PCBWAY
- C16: renamed from C_RES1; Assembly (none) -> YES; Supplier (none) -> PCBWAY
- C17: renamed from C_LREG1; Assembly (none) -> YES; Supplier (none) -> PCBWAY
- C18: renamed from C_RES2; Assembly (none) -> YES; Supplier (none) -> PCBWAY
- C2: renamed from C_MCU2; Assembly (none) -> YES; Supplier (none) -> PCBWAY
- C3: renamed from C_MCU_OSC1; Assembly (none) -> YES; Supplier (none) -> PCBWAY
- C4: renamed from C_MCU_OSC2; Assembly (none) -> YES; Supplier (none) -> PCBWAY
- C5: renamed from C_USB1; Assembly (none) -> YES; Supplier (none) -> PCBWAY
- C6: renamed from C_USB2; Assembly (none) -> YES; Supplier (none) -> PCBWAY
- C7: renamed from C_USB3; Assembly (none) -> YES; Supplier (none) -> PCBWAY
- C8: renamed from C_IN1; Assembly (none) -> YES; Supplier (none) -> PCBWAY
- C9: renamed from C_IN2; Assembly (none) -> YES; Supplier (none) -> PCBWAY
- CON1: renamed from CON_CTRL1; value Conn_01x04_Pin -> Conn_01x02_Pin; footprint Connector_PinHeader_2.54mm:PinHeader_1x04_P2.54mm_Horizontal -> custom_components:CON_2_pin; symbol Connector:Conn_01x04_Pin -> Connector:Conn_01x02_Pin; Assembly (none) -> NO; Supplier (none) -> GME; Supplier no. (none) -> 800-163; URL (none) -> https://www.gme.cz/v/1497299/kls-psh02-02pg-konektor-vidlic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
- CON4: renamed from CON_VIN1; footprint Connector_PinHeader_2.54mm:PinHeader_1x02_P2.54mm_Horizontal -> custom_components:CON_2_pin; Assembly (none) -> NO; Supplier (none) -> GME; Supplier no. (none) -> 800-163; URL (none) -> https://www.gme.cz/v/1497299/kls-psh02-02pg-konektor-vidlic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
- IC1: renamed from MCU1; value ATmega328PB-A -> ATmega328PB-AU; Assembly (none) -> YES; Supplier (none) -> LCSC; Supplier no. (none) -> C132230; URL (none) -> https://www.lcsc.com/product-detail/Microcontrollers-MCU-MP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
- IC2: renamed from UART-USB1; value FT231XS -> FT231XS-R; Assembly (none) -> YES; Supplier (none) -> LCSC; Supplier no. (none) -> C132160; URL (none) -> https://www.lcsc.com/product-detail/USB-Converters_FTDI-FT2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
- IC3: renamed from SCH1; Assembly (none) -> YES; Supplier (none) -> LCSC; Supplier no. (none) -> C5359730; URL (none) -> https://www.lcsc.com/product-detail/Inverters_Nexperia-74HC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
- IC4: renamed from LREG1; value LM78M05_TO252 -> L78M05ABDT-TR; Assembly (none) -> YES; Supplier (none) -> LCSC; Supplier no. (none) -> C58069; URL (none) -> https://www.lcsc.com/product-detail/Voltage-Regulators-span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
- LED1: renamed from LED_RX1; Assembly (none) -> YES; Supplier (none) -> PCBWAY
- LED2: renamed from LED_TX1; Assembly (none) -> YES; Supplier (none) -> PCBWAY
- LED3: renamed from LED_PWR1; Assembly (none) -> YES; Supplier (none) -> PCBWAY
- OPT1: renamed from OPTL1; Assembly (none) -> YES; Supplier (none) -> LCSC; Supplier no. (none) -> C17666883; URL (none) -> https://www.lcsc.com/product-detail/Transistor-Photovoltaic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
- OPT2: renamed from OPTR1; Assembly (none) -> YES; Supplier (none) -> LCSC; Supplier no. (none) -> C17666883; URL (none) -> https://www.lcsc.com/product-detail/Transistor-Photovoltaic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
- OSC1: renamed from OSC_MCU1; Assembly (none) -> YES; Supplier (none) -> LCSC; Supplier no. (none) -> C498200; URL (none) -> https://www.lcsc.com/product-detail/Crystals_span-style-bac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
- R10: renamed from R_IN2; Assembly (none) -> YES; Supplier (none) -> PCBWAY
- R11: renamed from R_IN3; Assembly (none) -> YES; Supplier (none) -> PCBWAY
- R12: renamed from R_RES1; Assembly (none) -> YES; Supplier (none) -> PCBWAY
- R13: renamed from RL1; Assembly (none) -> YES; Supplier (none) -> PCBWAY
- R14: renamed from RR1; Assembly (none) -> YES; Supplier (none) -> PCBWAY
- R15: renamed from R_RES2; Assembly (none) -> YES; Supplier (none) -> PCBWAY
- R16: renamed from R1; Assembly (none) -> YES; Supplier (none) -> PCBWAY
- R2, R3: Assembly (none) -> YES; Supplier (none) -> PCBWAY
- R4: renamed from R_USB1; Assembly (none) -> YES; Supplier (none) -> PCBWAY
- R5: renamed from R_USB2; Assembly (none) -> YES; Supplier (none) -> PCBWAY
- R6: renamed from R_IN4; Assembly (none) -> YES; Supplier (none) -> PCBWAY
- R7: renamed from R_IN5; Assembly (none) -> YES; Supplier (none) -> PCBWAY
- R8: renamed from R_IN6; Assembly (none) -> YES; Supplier (none) -> PCBWAY
- R9: renamed from R_IN1; Assembly (none) -> YES; Supplier (none) -> PCBWAY
- SW4: renamed from SW1; footprint Button_Switch_SMD:SW_SPST_B3U-1000P -> custom_components:switch; Assembly (none) -> YES; Supplier (none) -> LCSC; Supplier no. (none) -> C455280; URL (none) -> https://www.lcsc.com/product-detail/Tactile-Switches_XUNPU-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
- SW5: renamed from SW2; Assembly (none) -> NO; Supplier (none) -> GME; Supplier no. (none) -> 632-048; URL (none) -> https://www.gme.cz/v/1500415/ece-edg101s-dip-prepinac-1pol
Connections:
- net +12V: now also CON5.1 (Pin_1)
- net +5V: now also HDR1.2 (Pin_2), R1.2, RV1.3
- net DISPLAY_D0: now also IC1.15 (PB3), HDR1.11 (Pin_11); no longer IC1.17 (PB5)
- net DISPLAY_D1: now also IC1.14 (PB2), HDR1.12 (Pin_12); no longer IC1.16 (PB4)
- net DISPLAY_D2: now also IC1.13 (PB1), HDR1.13 (Pin_13); no longer IC1.15 (PB3)
- net DISPLAY_D3: now also IC1.12 (PB0), HDR1.14 (Pin_14); no longer IC1.14 (PB2)
- net DISPLAY_EN: now also IC1.16 (PB4), HDR1.6 (Pin_6); no longer IC1.13 (PB1)
- net DISPLAY_RS: now also IC1.17 (PB5), HDR1.4 (Pin_4); no longer IC1.12 (PB0)
- net GND: now also CON1.2 (Pin_2), IC1.2 (PD4), CON3.3 (Pin_3), CON5.2 (Pin_2), HDR1.1 (Pin_1), HDR1.16 (Pin_16), HDR1.5 (Pin_5), RV1.1, SW1.1, SW2.1, SW3.1; no longer CON1.1 (Pin_1), IC1.11 (PD7)
- net IN_LEFT: now also CON5.3 (Pin_3)
- net IN_RIGHT: now also CON5.4 (Pin_4)
- net RESET: now also IC1.11 (PD7); no longer IC1.10 (PD6)
- net START: now also IC1.9 (PD5); no longer IC1.2 (PD4)
- net STOP: now also IC1.10 (PD6); no longer IC1.9 (PD5)
- net USB_D+: now also CON3.2 (Pin_2)
- net USB_D-: now also CON3.1 (Pin_1)
- net at R11.1, R8.2: now also SW3.2; no longer CON1.4 (Pin_4)
- net at R6.2, R9.1: now also CON1.1 (Pin_1), SW1.2; no longer CON1.2 (Pin_2)
- net at R10.1, R7.2: now also SW2.2; no longer CON1.3 (Pin_3)
- new net: HDR1.15 (Pin_15), R1.1
- new net: HDR1.3 (Pin_3), RV1.2
- no-connect marks 8 -> 11

Commit message: final update2
Parts:
- CON2: footprint KLS_connector:16_pin -> custom_components:CON16_pin
Other:
- note added: "Display 16x2"
- moved on the sheet: HDR1, R1, RV1

Commit message: final
Parts:
- added CON6: AVR-ISP-6, Connector_IDC:IDC-Header_2x03_P2.54mm_Vertical, symbol Connector:AVR-ISP-6
Connections:
- net +5V: now also CON6.2 (VCC)
- net DISPLAY_D0: now also CON6.4 (MOSI)
- net DISPLAY_EN: now also CON6.1 (MISO)
- net DISPLAY_RS: now also CON6.3 (SCK)
- net GND: now also CON6.6 (GND)
- net RES: now also CON6.5 (~{RST})

Commit message: major changes, production ready
Parts:
- removed C12: 100nF, Capacitor_SMD:C_0603_1608Metric, symbol Device:C
- removed C13: 1nF, Capacitor_SMD:C_0603_1608Metric, symbol Device:C
- removed CON3: Conn_01x03, custom_components:CON_3_pin, symbol Connector_Generic:Conn_01x03
- removed OPT1, OPT2: TLP185xSE, Package_SO:SOIC-4_4.55x3.7mm_P2.54mm, symbol Isolator:TLP185xSE
- added CON3: Conn_01x04_Pin, custom_components:CON_4_pin, symbol Connector:Conn_01x04_Pin
- added D1, D2: BZX384-B5V1,115, Diode_SMD:D_SOD-323, symbol Device:D_Zener
- added Q1, Q2: PMBT3904,215, Package_TO_SOT_SMD:SOT-23, symbol Simulation_SPICE:NPN
- added R17, R18, R22: 10K, Resistor_SMD:R_0603_1608Metric, symbol Device:R
- added R19, R20: 1.2K, Capacitor_SMD:C_0603_1608Metric, symbol Device:R
- added R21: 4K7, Resistor_SMD:R_0603_1608Metric, symbol Device:R
- C1, C16, C17, C18, C2, C5: value 100nF -> 100nF, 16V
- C10, C8, C9: value 100n -> 100n, 16V
- C11: value 1uF -> 330nF, 25V
- C14, C15: value 100nF -> 1n, 25V
- C3, C4: value 22pF -> 22pF, 16V
- C6, C7: value 47pF -> 47pF, 16V
- IC1, IC2: Accept alternative part (none) -> NO
- IC3, IC4, OSC1, SW4: Accept alternative part (none) -> YES
- R13, R14: value 550R -> 1.2K; footprint Resistor_SMD:R_0603_1608Metric -> Capacitor_SMD:C_0603_1608Metric
Connections:
- net +12V: now also R14.2, R20.2
- net GND: now also CON3.4 (Pin_4), D1.2 (A), D2.2 (A), Q1.2 (E), Q2.2 (E), R22.2
- net USB_D+: now also CON3.2 (Pin_2)
- net USB_D-: now also CON3.3 (Pin_3)
- net at R14.1: now also R13.2; no longer C15.1
- net at R13.1: now also CON5.4 (Pin_4), D1.1 (K), R17.2; no longer C14.1
- net at R3.1: now also IC2.19 (CBUS3); no longer IC2.17 (CBUS1)
- net IN_LEFT: no longer names the net of CON5.3 (Pin_3)
- net IN_LEFT: now also D2.1 (K), R18.2, R19.1; no longer R13.2
- removed net IN_RIGHT: CON5.4 (Pin_4), R14.2
- net OPTL renamed LEFT
- net LEFT: now also Q1.3 (C)
- net OPTR renamed RIGHT
- net RIGHT: now also Q2.3 (C)
- new net: C14.1, Q1.1 (B), R18.1
- new net: R19.2, R20.1
- new net: C15.1, Q2.1 (B), R17.1
- new net: CON3.1 (Pin_1), R21.1
- new net VBUS_SENSE: IC2.17 (CBUS1), R21.2, R22.1
- no-connect marks 11 -> 10
Other:
- moved on the sheet: C11, CON4, CON5, LED1, R2

Commit message: panelization
Parts:
- R16, R2, R3: value 330R -> 1K
- SW4: value SW_Push -> SW_Push_SMD
Changed lines of the file:
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@@
 			)
 		)
-		(property "Value" "330R"
+		(property "Value" "1K"
 			(at 269.24 34.2899 0)
 			(effects
@@
 			)
 		)
-		(property "Value" "SW_Push"
+		(property "Value" "SW_Push_SMD"
 			(at 250.19 148.5899 90)
 			(effects
@@
 			)
 		)
-		(property "Value" "330R"
+		(property "Value" "1K"
 			(at 49.53 38.608 90)
 			(effects
@@
 			)
 		)
-		(property "Value" "330R"
+		(property "Value" "1K"
 			(at 49.53 30.226 90)
 			(effects

Commit message: update
Parts:
- IC2: value FT231XS-R -> FT231XS-R
- IC3: value 74HC3G14DP,125 -> 74HC3G14DP,125
Changed lines of the file:
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@@
 (kicad_sch
-	(version 20231120)
+	(version 20250114)
 	(generator "eeschema")
-	(generator_version "8.0")
+	(generator_version "9.0")
 	(paper "A4")
 	(title_block
@@
 		(rev "1.0")
 	)
+	(rectangle
+		(start 30.48 13.97)
+		(end 182.88 73.66)
+		(stroke
+			(width 0)
+			(type default)
+		)
+		(fill
+			(type none)
+		)
+	)
+	(rectangle
+		(start 190.5 59.69)
+		(end 270.51 111.76)
+		(stroke
+			(width 0)
+			(type default)
+		)
+		(fill
+			(type none)
+		)
+	)
+	(rectangle
+		(start 220.98 113.03)
+		(end 280.67 161.29)
+		(stroke
+			(width 0)
+			(type default)
+		)
+		(fill
+			(type none)
+		)
+	)
+	(rectangle
+		(start 186.69 13.97)
+		(end 280.67 55.88)
+		(stroke
+			(width 0)
+			(type default)
+		)
+		(fill
+			(type none)
+		)
+	)
+	(text "Reset"
+		(exclude_from_sim no)
+		(at 254.762 118.872 0)
+		(effects
+			(font
+				(size 5 5)
+			)
+		)
+	)
+	(text "Button inputs"
+		(exclude_from_sim no)
+		(at 146.05 150.622 0)
+		(effects
+			(font
+				(size 5 5)
+			)
+		)
+	)
+	(text "USB to serial"
+		(exclude_from_sim no)
+		(at 142.748 66.294 0)
+		(effects
+			(font
+				(size 5 5)
+			)
+		)
+	)
+	(text "Target inputs"
+		(exclude_from_sim no)
+		(at 216.408 107.442 0)
+		(effects
+			(font
+				(size 5 5)
+			)
+		)
+	)
+	(text "Display 16x2"
+		(exclude_from_sim no)
+		(at 71.12 112.522 0)
+		(effects
+			(font
+				(size 5 5)
+			)
+		)
+	)
+	(text "Power"
+		(exclude_from_sim no)
+		(at 209.804 49.276 0)
+		(effects
+			(font
+				(size 5 5)
+			)
+		)
+	)
+	(text_box ""
+		(exclude_from_sim no)
+		(at 41.91 76.2 0)
+		(size 71.12 41.91)
+		(margins 0.9525 0.9525 0.9525 0.9525)
+		(stroke
+			(width 0)
+			(type default)
+		)
+		(fill
+			(type none)
+		)
+		(effects
+			(font
+				(size 1.27 1.27)
+			)
+			(justify left top)
+		)
+	)
+	(text_box ""
+		(exclude_from_sim no)
+		(at 116.84 74.93 0)
+		(size 71.12 81.28)
+		(margins 0.9525 0.9525 0.9525 0.9525)
+		(stroke
+			(width 0)
+			(type default)
+		)
+		(fill
+			(type none)
+		)
+		(effects
+			(font
+				(size 1.27 1.27)
+			)
+			(justify left top)
+		)
+	)
 	(junction
 		(at 25.4 85.09)
@@
 		)
 	)
-	(rectangle
-		(start 30.48 13.97)
-		(end 182.88 73.66)
-		(stroke
-			(width 0)
-			(type default)
-		)
-		(fill
-			(type none)
-		)
-	)
-	(rectangle
-		(start 190.5 59.69)
-		(end 270.51 111.76)
-		(stroke
-			(width 0)
-			(type default)
-		)
-		(fill
-			(type none)
-		)
-	)
-	(rectangle
-		(start 220.98 113.03)
-		(end 280.67 161.29)
-		(stroke
-			(width 0)
-			(type default)
-		)
-		(fill
-			(type none)
-		)
-	)
-	(rectangle
-		(start 186.69 13.97)
-		(end 280.67 55.88)
-		(stroke
-			(width 0)
-			(type default)
-		)
-		(fill
-			(type none)
-		)
-	)
-	(text_box ""
-		(exclude_from_sim no)
-		(at 41.91 76.2 0)
-		(size 71.12 41.91)
-		(stroke
-			(width 0)
-			(type default)
-		)
-		(fill
-			(type none)
-		)
-		(effects
-			(font
-				(size 1.27 1.27)
-			)
-			(justify left top)
-		)
-	)
-	(text_box ""
-		(exclude_from_sim no)
-		(at 116.84 74.93 0)
-		(size 71.12 81.28)
-		(stroke
-			(width 0)
-			(type default)
-		)
-		(fill
-			(type none)
-		)
-		(effects
-			(font
-				(size 1.27 1.27)
-			)
-			(justify left top)
-		)
-	)
-	(text "Reset"
-		(exclude_from_sim no)
-		(at 254.762 118.872 0)
-		(effects
-			(font
-				(size 5 5)
-			)
-		)
-	)
-	(text "Button inputs"
-		(exclude_from_sim no)
-		(at 146.05 150.622 0)
-		(effects
-			(font
-				(size 5 5)
-			)
-		)
-	)
-	(text "USB to serial"
-		(exclude_from_sim no)
-		(at 142.748 66.294 0)
-		(effects
-			(font
-				(size 5 5)
-			)
-		)
-	)
-	(text "Target inputs"
-		(exclude_from_sim no)
-		(at 216.408 107.442 0)
-		(effects
-			(font
-				(size 5 5)
-			)
-		)
-	)
-	(text "Display 16x2"
-		(exclude_from_sim no)
-		(at 71.12 112.522 0)
-		(effects
-			(font
-				(size 5 5)
-			)
-		)
-	)
-	(text "Power"
-		(exclude_from_sim no)
-		(at 209.804 49.276 0)
-		(effects
-			(font
-				(size 5 5)
-			)
-		)
-	)
 	(label "USB_D-"
 		(at 121.92 45.72 0)
-		(fields_autoplaced yes)
 		(effects
 			(font
@@
 	(label "USB_D+"
 		(at 121.92 48.26 0)
-		(fields_autoplaced yes)
 		(effects
 			(font
@@
 			)
 		)
-		(property "Value" "74HC3G14DP,125 "
+		(property "Value" "74HC3G14DP,125"
 			(at 168.91 101.6 0)
 			(effects
@@
 			)
 		)
-		(property "Value" "FT231XS-R "
+		(property "Value" "FT231XS-R"
 			(at 97.028 43.434 0)
 			(effects
@@
 		)
 	)
+	(embedded_fonts no)
 )
