File: PCB/FT_TargetSwitch/FT_TargetSwitch.kicad_sch (KiCad schematic)
At the start: 11 parts

Commit message: changed hall, switch
Parts:
- R_PUP1: footprint Resistor_SMD:R_0603_1608Metric_Pad0.98x0.95mm_HandSolder -> Resistor_SMD:R_1206_3216Metric_Pad1.30x1.75mm_HandSolder
Changed lines of the file:
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@@
 			)
 		)
-		(property "Footprint" "Resistor_SMD:R_0603_1608Metric_Pad0.98x0.95mm_HandSolder"
+		(property "Footprint" "Resistor_SMD:R_1206_3216Metric_Pad1.30x1.75mm_HandSolder"
 			(at 90.932 83.82 90)
 			(effects

Commit message: update pcbs
Parts:
- removed D1, D2: M7, Diode_SMD:D_SMA_Handsoldering, symbol Device:D
- removed SW_L1, SW_R1: SW_DIP_x02, Button_Switch_THT:SW_DIP_SPSTx02_Slide_9.78x7.26mm_W7.62mm_P2.54mm, symbol Switch:SW_DIP_x02
- R_PUP1: footprint Resistor_SMD:R_1206_3216Metric_Pad1.30x1.75mm_HandSolder -> Resistor_SMD:R_0603_1608Metric
Connections:
- net L_OUT is gone; now on net OUT: CON_IO1.3 (Pin_3)
- net Q_UOT_DRAIN is gone; now on net OUT: Q_OUT1.3 (D)
- net R_OUT is gone; now on net PASSTHRU_OUT: CON_IO1.4 (Pin_4)
- net PASTRHRU_IN renamed PASSTHRU_OUT

Commit message: final
Parts:
- CON1: renamed from CON_IO1; Assembly (none) -> NO; Supplier (none) -> GME; Supplier no. (none) -> 800-170; URL (none) -> https://www.gme.cz/v/1497969/kls-psh02-04pg-konektor-vidlic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
- CON2: renamed from CON_PASTHRU1; Assembly (none) -> NO; Supplier (none) -> GME; Supplier no. (none) -> 800-164; URL (none) -> https://www.gme.cz/v/1497964/kls-psh02-03pg-konektor-vidlic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
- CON3: renamed from CON_HAL1; Assembly (none) -> NO; Supplier (none) -> GME; Supplier no. (none) -> 800-164; URL (none) -> https://www.gme.cz/v/1497964/kls-psh02-03pg-konektor-vidlic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
- CON4: renamed from CON_LED1; Assembly (none) -> NO; Supplier (none) -> GME; Supplier no. (none) -> 800-163; URL (none) -> https://www.gme.cz/v/1497299/kls-psh02-02pg-konektor-vidlic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
- Q1: renamed from Q_OUT1; Assembly (none) -> YES; Supplier (none) -> LCSC; Supplier no. (none) -> C2592; URL (none) -> https://www.lcsc.com/product-detail/MOSFETs_Infineon-Techno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
- Q2: renamed from Q_LED1; Assembly (none) -> YES; Supplier (none) -> LCSC; Supplier no. (none) -> C2585; URL (none) -> https://www.lcsc.com/product-detail/MOSFETs_Infineon-Techno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
- R1: renamed from R_PUP1; value 100K -> 10K; Assembly (none) -> YES; Supplier (none) -> PCBWAY

Commit message: major changes, production ready
Parts:
- removed Q1: IRLML5203, Package_TO_SOT_SMD:SOT-23, symbol Transistor_FET:IRLML5203
- added F1: BSMD0603-025-12V, Fuse:Fuse_0603_1608Metric, symbol Device:Polyfuse
- added Q1: 2N7002,215, Package_TO_SOT_SMD:SOT-23, symbol Simulation_SPICE:NMOS
- Q2: Accept alternative part (none) -> YES
Connections:
- net +12V: now also F1.2; no longer CON1.1 (Pin_1), CON2.1 (Pin_1)
- net GND: now also Q1.2 (S)
- net HAL_IN: now also Q1.1 (G)
- net OUT: now also CON1.1 (Pin_1), CON2.1 (Pin_1), F1.1, Q1.3 (D)
- net PASSTHRU_OUT renamed PASSTHRU
Other:
- moved on the sheet: CON1, CON2, CON3, CON4

Commit message: panelization
Parts:
- renumbered CON1 to CON201, CON2 to CON202, CON3 to CON203, CON4 to CON204, F1 to F201, Q1 to Q201, Q2 to Q202, R1 to R201
Changed lines of the file:
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@@
 		(on_board yes)
 		(dnp no)
-		(property "Reference" "R1"
+		(property "Reference" "R201"
 			(at 94.234 82.55 0)
 			(effects
@@
 			(project "FT_TargetSwitch"
 				(path "/135d114f-f68d-4e79-9ee5-cca5273d2aa9"
-					(reference "R1")
+					(reference "R201")
 					(unit 1)
 				)
@@
 		(on_board yes)
 		(dnp no)
-		(property "Reference" "Q1"
+		(property "Reference" "Q201"
 			(at 82.042 90.17 0)
 			(effects
@@
 			(project "FT_TargetSwitch"
 				(path "/135d114f-f68d-4e79-9ee5-cca5273d2aa9"
-					(reference "Q1")
+					(reference "Q201")
 					(unit 1)
 				)
@@
 		(dnp no)
 		(fields_autoplaced yes)
-		(property "Reference" "CON2"
+		(property "Reference" "CON202"
 			(at 68.58 125.73 90)
 			(effects
@@
 			(project "FT_TargetSwitch"
 				(path "/135d114f-f68d-4e79-9ee5-cca5273d2aa9"
-					(reference "CON2")
+					(reference "CON202")
 					(unit 1)
 				)
@@
 		(dnp no)
 		(fields_autoplaced yes)
-		(property "Reference" "CON3"
+		(property "Reference" "CON203"
 			(at 90.17 125.73 90)
 			(effects
@@
 			(project "FT_TargetSwitch"
 				(path "/135d114f-f68d-4e79-9ee5-cca5273d2aa9"
-					(reference "CON3")
+					(reference "CON203")
 					(unit 1)
 				)
@@
 		(on_board yes)
 		(dnp no)
-		(property "Reference" "F1"
+		(property "Reference" "F201"
 			(at 77.724 106.426 90)
 			(effects
@@
 			(project "FT_TargetSwitch"
 				(path "/135d114f-f68d-4e79-9ee5-cca5273d2aa9"
-					(reference "F1")
+					(reference "F201")
 					(unit 1)
 				)
@@
 		(on_board yes)
 		(dnp no)
-		(property "Reference" "CON1"
+		(property "Reference" "CON201"
 			(at 42.926 126.238 90)
 			(effects
@@
 			(project "FT_TargetSwitch"
 				(path "/135d114f-f68d-4e79-9ee5-cca5273d2aa9"
-					(reference "CON1")
+					(reference "CON201")
 					(unit 1)
 				)
@@
 		(on_board yes)
 		(dnp no)
-		(property "Reference" "Q2"
+		(property "Reference" "Q202"
 			(at 104.14 89.916 0)
 			(effects
@@
 			(project "FT_TargetSwitch"
 				(path "/135d114f-f68d-4e79-9ee5-cca5273d2aa9"
-					(reference "Q2")
+					(reference "Q202")
 					(unit 1)
 				)
@@
 		(on_board yes)
 		(dnp no)
-		(property "Reference" "CON4"
+		(property "Reference" "CON204"
 			(at 99.568 125.73 90)
 			(effects
@@
 			(project "FT_TargetSwitch"
 				(path "/135d114f-f68d-4e79-9ee5-cca5273d2aa9"
-					(reference "CON4")
+					(reference "CON204")
 					(unit 1)
 				)

Commit message: update
Connections:
- net OUT: no longer CON201.1 (Pin_1), CON202.1 (Pin_1), F201.1
- new net: CON201.1 (Pin_1), CON202.1 (Pin_1), F201.1
Changed lines of the file:
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@@
 (kicad_sch
-	(version 20231120)
+	(version 20250114)
 	(generator "eeschema")
-	(generator_version "8.0")
+	(generator_version "9.0")
 	(paper "A4")
 	(junction
@@
 	(wire
 		(pts
+			(xy 39.37 109.22) (xy 39.37 118.11)
+		)
+		(stroke
+			(width 0)
+			(type default)
+		)
+	)
+	(wire
+		(pts
+			(xy 71.12 105.41) (xy 71.12 118.11)
+		)
+		(stroke
+			(width 0)
+			(type default)
+		)
+	)
+	(wire
+		(pts
+			(xy 82.55 109.22) (xy 87.63 109.22)
+		)
+		(stroke
+			(width 0)
+			(type default)
+		)
+	)
+	(wire
+		(pts
+			(xy 80.01 113.03) (xy 90.17 113.03)
+		)
+		(stroke
+			(width 0)
+			(type default)
+		)
+	)
+	(wire
+		(pts
+			(xy 92.71 77.47) (xy 101.6 77.47)
+		)
+		(stroke
+			(width 0)
+			(type default)
+		)
+	)
+	(wire
+		(pts
+			(xy 92.71 77.47) (xy 92.71 80.01)
+		)
+		(stroke
+			(width 0)
+			(type default)
+		)
+	)
+	(wire
+		(pts
+			(xy 90.17 113.03) (xy 104.14 113.03)
+		)
+		(stroke
+			(width 0)
+			(type default)
+		)
+	)
+	(wire
+		(pts
+			(xy 44.45 100.33) (xy 85.09 100.33)
+		)
+		(stroke
+			(width 0)
+			(type default)
+		)
+	)
+	(wire
+		(pts
+			(xy 68.58 113.03) (xy 80.01 113.03)
+		)
+		(stroke
+			(width 0)
+			(type default)
+		)
+	)
+	(wire
+		(pts
+			(xy 104.14 118.11) (xy 104.14 113.03)
+		)
+		(stroke
+			(width 0)
+			(type default)
+		)
+	)
+	(wire
+		(pts
+			(xy 87.63 118.11) (xy 87.63 109.22)
+		)
+		(stroke
+			(width 0)
+			(type default)
+		)
+	)
+	(wire
+		(pts
+			(xy 92.71 91.44) (xy 93.98 91.44)
+		)
+		(stroke
+			(width 0)
+			(type default)
+		)
+	)
+	(wire
+		(pts
+			(xy 66.04 109.22) (xy 72.39 109.22)
+		)
+		(stroke
+			(width 0)
+			(type default)
+		)
+	)
+	(wire
+		(pts
+			(xy 85.09 100.33) (xy 85.09 96.52)
+		)
+		(stroke
+			(width 0)
+			(type default)
+		)
+	)
+	(wire
+		(pts
+			(xy 46.99 105.41) (xy 71.12 105.41)
+		)
+		(stroke
+			(width 0)
+			(type default)
+		)
+	)
+	(wire
+		(pts
 			(xy 39.37 109.22) (xy 66.04 109.22)
 		)
@@
 	(wire
 		(pts
-			(xy 39.37 109.22) (xy 39.37 118.11)
-		)
-		(stroke
-			(width 0)
-			(type default)
-		)
-	)
-	(wire
-		(pts
-			(xy 71.12 105.41) (xy 71.12 118.11)
-		)
-		(stroke
-			(width 0)
-			(type default)
-		)
-	)
-	(wire
-		(pts
-			(xy 82.55 109.22) (xy 87.63 109.22)
-		)
-		(stroke
-			(width 0)
-			(type default)
-		)
-	)
-	(wire
-		(pts
-			(xy 80.01 113.03) (xy 90.17 113.03)
-		)
-		(stroke
-			(width 0)
-			(type default)
-		)
-	)
-	(wire
-		(pts
-			(xy 92.71 77.47) (xy 101.6 77.47)
-		)
-		(stroke
-			(width 0)
-			(type default)
-		)
-	)
-	(wire
-		(pts
-			(xy 92.71 77.47) (xy 92.71 80.01)
-		)
-		(stroke
-			(width 0)
-			(type default)
-		)
-	)
-	(wire
-		(pts
-			(xy 90.17 113.03) (xy 104.14 113.03)
-		)
-		(stroke
-			(width 0)
-			(type default)
-		)
-	)
-	(wire
-		(pts
-			(xy 44.45 100.33) (xy 85.09 100.33)
-		)
-		(stroke
-			(width 0)
-			(type default)
-		)
-	)
-	(wire
-		(pts
-			(xy 68.58 113.03) (xy 80.01 113.03)
-		)
-		(stroke
-			(width 0)
-			(type default)
-		)
-	)
-	(wire
-		(pts
-			(xy 104.14 118.11) (xy 104.14 113.03)
-		)
-		(stroke
-			(width 0)
-			(type default)
-		)
-	)
-	(wire
-		(pts
-			(xy 87.63 118.11) (xy 87.63 109.22)
-		)
-		(stroke
-			(width 0)
-			(type default)
-		)
-	)
-	(wire
-		(pts
-			(xy 92.71 91.44) (xy 93.98 91.44)
-		)
-		(stroke
-			(width 0)
-			(type default)
-		)
-	)
-	(wire
-		(pts
-			(xy 66.04 109.22) (xy 72.39 109.22)
-		)
-		(stroke
-			(width 0)
-			(type default)
-		)
-	)
-	(wire
-		(pts
-			(xy 85.09 100.33) (xy 85.09 96.52)
-		)
-		(stroke
-			(width 0)
-			(type default)
-		)
-	)
-	(wire
-		(pts
-			(xy 46.99 105.41) (xy 71.12 105.41)
-		)
-		(stroke
-			(width 0)
-			(type default)
-		)
-	)
-	(wire
-		(pts
 			(xy 46.99 105.41) (xy 46.99 118.11)
 		)
@@
 	(wire
 		(pts
+			(xy 101.6 96.52) (xy 101.6 118.11)
+		)
+		(stroke
+			(width 0)
+			(type default)
+		)
+	)
+	(wire
+		(pts
+			(xy 85.09 77.47) (xy 85.09 86.36)
+		)
+		(stroke
+			(width 0)
+			(type default)
+		)
+	)
+	(wire
+		(pts
 			(xy 44.45 100.33) (xy 44.45 118.11)
-		)
-		(stroke
-			(width 0)
-			(type default)
-		)
-	)
-	(wire
-		(pts
-			(xy 101.6 96.52) (xy 101.6 118.11)
-		)
-		(stroke
-			(width 0)
-			(type default)
-		)
-	)
-	(wire
-		(pts
-			(xy 85.09 77.47) (xy 85.09 86.36)
 		)
 		(stroke
@@
 	(label "PASSTHRU"
 		(at 53.34 105.41 0)
-		(fields_autoplaced yes)
 		(effects
 			(font
@@
 	(label "Q_UOT_DRAIN"
 		(at 85.09 100.33 180)
-		(fields_autoplaced yes)
 		(effects
 			(font
@@
 	(label "LED_OUT"
 		(at 101.6 99.06 180)
-		(fields_autoplaced yes)
 		(effects
 			(font
@@
 	)
 	(label "OUT"
-		(at 44.45 109.22 90)
-		(fields_autoplaced yes)
+		(at 44.45 106.68 90)
 		(effects
 			(font
@@
 	(label "HAL_IN"
 		(at 92.71 105.41 90)
-		(fields_autoplaced yes)
 		(effects
 			(font
@@
 		)
 	)
+	(embedded_fonts no)
 )
